File: Boards/LV Interface/LV Interface.sch (KiCad schematic (older format))
At the start: 18 parts, among them J1 Ampseal_35_VT, J10 MM_M_VT_20, J11 MicroFit_VT_4, J2 Ampseal_14_VT, J3 MicroFit_VT_4, J4 MM_M_VT_20, J6 MM_M_VT_20, J7 MM_M_VT_20, J8 UF_2_VT, J9 MM_M_VT_20, K1 G5Q-1A4-DC5-5V, U1 RJ45_VT, U2 Fuse_Holder_Blade, U3 Fuse_Holder_Blade

Commit message: First Layout Changes
Parts:
- added U4: Fuse_Holder_Blade, footprints:Fuse_Block_Holder, symbol formula:Fuse_Holder_Blade
- added U5: INA260, Package_SO:TSSOP-16_4.4x5mm_P0.65mm, symbol formula:INA260
- gave numbers to parts that had none: 3
Connections:
- net 12V: now also U4.1, U5.14 (IN-), U5.15 (IN-), U5.16 (IN-); no longer U2.2
- net CAN HIGH: now also J12.3, J2.10, J5.4; no longer J2.4, J5.3
- net CAN LOW: now also J12.4, J2.11, J5.5; no longer J2.5, J5.4
- net CS_GLV: now also J12.10, J5.11; no longer J12.6, J5.10
- net GND: now also J12.11, J12.12, J12.13, J12.14, J12.15, J12.16, J12.17, J12.18, J12.19, J12.20, J2.12, J2.5, J5.12, J5.13, J5.14, J5.15, J5.16, J5.17, J5.18, J5.19, J5.20, J6.20, U6.4 (A1), U5.11 (GND), U5.4 (A1), U5.5 (A0), U5.6 (GND); no longer J1.30, J2.9
- net MC TEMP +: now also J6.10; no longer J6.15
- net MC TEMP -: now also J2.7, J6.11; no longer J2.8, J6.17
- net MISO_GLV: now also J12.7, J5.8; no longer J12.3, J5.7
- net MOSI_GLV: now also J12.8, J5.9; no longer J12.4, J5.8
- net MOTOR TEMP +: now also J6.8; no longer J6.9
- net MOTOR TEMP -: now also J2.2, J6.9; no longer J2.3, J6.11
- net RADIATOR TEMP +: now also J2.8; no longer J2.10
- net RADIATOR TEMP -: now also J2.9, J6.7; no longer J2.12, J6.8
- net SCK_GLV: now also J12.9, J5.10; no longer J12.5, J5.9
- net SCL_GLV: now also J12.5, J5.6, U6.9 (SCL), U5.9 (SCL); no longer J12.7, J5.11
- net SDA_GLV: now also J12.6, J5.7, U6.8 (SDA), U5.8 (SDA); no longer J12.8, J5.12
- net 12V_Cooling_Fused: now reaches U6.1 (IN+), U6.2 (IN+), U6.3 (IN+)
- net 12V_Cooling_Fused: now also U6.12 (VBUS), U4.2
- net 5V_GLV: now reaches U6.10 (VS)
- net 5V_GLV: now also J5.3, U6.5 (A0), U5.10 (VS)
- net 12V_Cooling: now reaches U6.14 (IN-), U6.15 (IN-), U6.16 (IN-)
- net 12V_Cooling: now also J1.30
- net ALERT_GLV: now reaches U6.7 (ALERT)
- net ALERT_GLV: now also U5.7 (ALERT)
- net MC PRESSURE + renamed EXTRA TEMP 1 +
- net EXTRA TEMP 1 +: now also J6.12; no longer J6.18
- net MC PRESSURE - renamed EXTRA TEMP 2 +
- net EXTRA TEMP 2 +: now also J6.14; no longer J6.20
- net MC PRESSURE SENSE renamed EXTRA TEMP 1 -
- net EXTRA TEMP 1 -: now also J6.13; no longer J6.19
- net MC TEMP SENSE renamed EXTRA TEMP 3 +
- net EXTRA TEMP 3 +: now also J1.7; no longer J2.7
- removed net MOTOR TEMP SENSE: J2.2, J6.10
- net PUMP PRESSURE + renamed EXTRA TEMP 2 -
- net EXTRA TEMP 2 -: now also J6.15; no longer J6.12
- net PUMP PRESSURE - renamed EXTRA TEMP 3 -
- net EXTRA TEMP 3 -: now also J6.17; no longer J6.14
- removed net PUMP PRESSURE SENSE: J1.7, J6.13
- removed net RADIATOR TEMP SENSE: J2.11, J6.7
- new net 12V_Fused: U2.2, U5.1 (IN+), U5.12 (VBUS), U5.2 (IN+), U5.3 (IN+)
- new net EXTRA TEMP 4 +: J2.3, J6.18
- new net EXTRA TEMP 4 -: J2.4, J6.19
Other:
- note added: "Cooling Gas Guage\n\n"
- note added: "GLV Gas Guage\n\n"
- moved on the sheet: J12, J5, J8, U2, U3, U6

Commit message: Saving work
Parts:
- added J13: UF_2_VT, footprints:Ultrafit_2, symbol formula:UF_2_VT
- J2: footprint footprints:Ampseal_14 -> (none)
- U1: symbol formula:RJ45_VT -> LV-Interface-rescue:RJ45_VT-formula
- U2, U3, U4: footprint footprints:Fuse_Block_Holder -> (none)
Connections:
- net 12V: no longer J1.31, U4.1
- net GND: now also J13.2
- net 12V_Cooling renamed 12V_Cooling_Out
- new net COOLING PUMP +: J1.31, J13.1, U4.1
Other:
- note added: "Cooling\n Batt \n"
- note added: "GLV Batt \n"
- moved on the sheet: J11, J3, J8, U5, U6
