File: Boards/LV Interface/_autosave-LV Interface.kicad_pcb (KiCad board)
At the start: 4 copper layers, 20 parts, among them J1 Ampseal_35_VT, J10 MM_M_VT_20, J11 MicroFit_VT_4, J12 MM_F_RA_20, J2 Ampseal_14_VT, J3 MicroFit_VT_4, J4 MM_M_VT_20, J5 MM_F_RA_20, J6 MM_M_VT_20, J7 MM_M_VT_20, J8 UF_2_VT, J9 MM_M_VT_20, K1 G5Q-1A4-DC5-5V, U1 RJ45_VT, U2 Fuse_Holder_Blade, U3 Fuse_Holder_Blade, U4 Fuse_Holder_Blade, U5 INA260, U6 INA260

Commit message: Saving work
Parts:
- added J13: UF_2_VT, footprints:Ultrafit_2, F.Cu at (72.3, 72.4)
- U1: moved to B.Cu
- moved J2 111.5 mm to (55.0, 104.5)
- moved J11 106.0 mm to (50.1, 129.8)
- moved J8 106.0 mm to (42.6, 146.0)
- moved U6 106.0 mm to (41.8, 129.7)
- moved J6 80.4 mm to (141.9, 113.6), turned to 270 degrees
- moved J10 73.3 mm to (141.5, 103.0), turned to 270 degrees
- moved J12 71.1 mm to (141.6, 90.3), turned to 270 degrees
- moved J4 60.2 mm to (141.4, 53.0), turned to 270 degrees
- moved J9 54.1 mm to (141.4, 64.8), turned to 270 degrees
- moved J5 51.5 mm to (141.9, 77.5), turned to 270 degrees
- moved J7 48.5 mm to (141.3, 39.6), turned to 270 degrees
- moved U5 47.5 mm to (73.3, 117.0)
- moved J3 47.5 mm to (73.2, 107.3)
- moved U1 39.3 mm to (139.4, 31.9), turned to 180 degrees
Connections:
- net /12V_Cooling renamed /12V_Cooling_Out
- J1 pad 31: /12V -> /COOLING PUMP +
- U4 pad 1: /12V -> /COOLING PUMP +
Other:
- board outline added: 165.1 x 127 mm
- board text added: "For Instructional Use Only."
- board text added: "SOLIDWORKS Educational Product."
